File: hardware/photoframe.brd (EAGLE design)
At the start: 99.4 x 99.8 mm, 76 parts, among them J2 XF2L-3035-1, U0 EP4CE15E22, U4 MT48LC16M16A2, U5 OSCILLATOR5X3-PIN1-INDICATED, U6 AT25SF041-SOIC8, X1 1503_02

Commit message: add new board
Parts:
- removed C12: (no value), SparkFun-Passives:0402-CAP
- C45: device SparkFun-Passives:0402-CAP -> SparkFun-Passives:0805
- R3, R4: device SparkFun-Passives:0603-RES -> SparkFun-Passives:0402-RES
- moved C5 80.4 mm to (80.6, 45.6)
- moved C6 80.4 mm to (81.1, 47.9)
- moved D6 80.4 mm to (80.6, 42.6)
- moved R6 80.4 mm to (79.8, 40.4)
- moved C8 78.9 mm to (92.7, 46.0), flipped to the top, turned to 90 degrees
- moved C7 77.6 mm to (92.8, 40.8)
- moved D2 76.6 mm to (84.2, 50.1)
- moved D1 73.7 mm to (81.2, 51.9)
- moved U2 53.0 mm to (50.2, 50.8), turned to 0 degrees
- moved D5 52.7 mm to (33.5, 8.50), turned to 315 degrees
- moved R5 52.2 mm to (32.2, 6.50), turned to 135 degrees
- moved C4 44.1 mm to (38.8, 10.2), turned to 45 degrees
- moved /RST 42.3 mm to (108.7, 35.0)
- moved GND 42.3 mm to (112.7, 35.0)
- moved IRQ 42.3 mm to (110.7, 35.0)
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Connections:
- removed net CKE: U0.133, U4.37
- removed net CS: U0.85, U4.19
- removed net N$12: S1.3, S1.4, U0.128
- new net N$16: U0.32
- net /RST: no longer U0.32
- net 1.0V: no longer C12.1
- net 3.3V: now also U4.37; no longer U0.96
- net A0: now also U0.67; no longer U0.76
- net A1: now also U0.66; no longer U0.69
- net A10: now also U0.68; no longer U0.77
- net A2: now also U0.65; no longer U0.68
- net A3: now also U0.64; no longer U0.67
- net BA0: now also U0.71; no longer U0.83
- net BA1: now also U0.69; no longer U0.80
- net CAS: now also U0.76; no longer U0.99
- net CLK: now also U0.133; no longer U0.132
- net CLK+: now also U0.59; no longer U0.50
- net CLK-: now also U0.60; no longer U0.51
- net DQ0: now also U0.100; no longer U0.11
- net DQ1: now also U0.104; no longer U0.10
- net DQ10: now also U0.120; no longer U0.119
- net DQ11: now also U0.119; no longer U0.111
- net DQ12: now also U0.115; no longer U0.112
- net DQ13: now also U0.114; no longer U0.113
- net DQ14: now also U0.113; no longer U0.114
- net DQ15: now also U0.112; no longer U0.115
- net DQ2: now also U0.105; no longer U0.7
- net DQ3: now also U0.106; no longer U0.110
- net DQ4: now also U0.110; no longer U0.106
- net DQ5: now also U0.111; no longer U0.105
- net DQ6: now also U0.85; no longer U0.104
- net DQ7: now also U0.83; no longer U0.103
- net DQ8: now also U0.125; no longer U0.121
- net DQ9: now also U0.121; no longer U0.120
- net DQMH: now also U0.132; no longer U0.125
- net DQML: now also U0.80; no longer U0.101
- net GND: now also U4.19; no longer C12.2, U0.94, U0.97
- net IN0+: now also U0.103; no longer U0.87
- net IN0-: now also U0.101; no longer U0.86
- net IN1+: now also U0.99; no longer U0.71
- net IN1-: now also U0.98; no longer U0.72
- net IN2+: now also U0.87; no longer U0.59
- net IN2-: now also U0.86; no longer U0.60
- net IN3+: now also U0.50; no longer U0.43
- net IN3-: now also U0.51; no longer U0.44
- net IRQ: no longer U0.129
- net LED_PWM: no longer U0.46
- net N$10: now also S1.3, S1.4, U0.129; no longer D1.C, U0.39
- net RAS: now also U0.72; no longer U0.98
- net SCL: no longer U0.31
- net SDA: no longer U0.30
- net SDCD: no longer U0.127
- net SDCLK: now also U0.28; no longer U0.61
- net SDCMD: now also U0.11; no longer U0.64
- net SDD0: now also U0.30; no longer U0.58
- net SDD1: now also U0.31; no longer U0.49
- net SDD2: now also U0.7; no longer U0.66
- net SDD3: now also U0.10; no longer U0.65
- net UART_RX: now also U0.58; no longer U0.54
- net UART_TX: now also U0.61; no longer U0.42
- net WE: now also U0.77; no longer U0.100
Routing:
- net 3.3V: track 325.3 -> 199.9 mm, vias 33 -> 24
- net SDD1: track 106.9 -> 37.4 mm
- net SDD0: track 99.9 -> 37.0 mm
- net SDCMD: track 89.3 -> 29.4 mm
- net /RST: track 58.3 -> 0.00 mm, vias 2 -> 0
- net SDCLK: track 94.3 -> 36.6 mm
- net SDD3: track 86.2 -> 29.0 mm
- net SDD2: track 83.2 -> 27.9 mm
- net SCL: track 53.2 -> 0.00 mm, vias 4 -> 0
- net SDA: track 50.1 -> 0.00 mm, vias 4 -> 0
- net 1.0V: track 169.4 -> 123.2 mm, vias 18 -> 9
- net IRQ: track 40.2 -> 0.00 mm, vias 2 -> 0
- net CKE: track 30.9 -> 0.00 mm
- net CS: track 30.8 -> 0.00 mm
- net UART_TX: track 48.5 -> 20.5 mm, vias 1 -> 0
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