File: hardware/photoframe.sch (EAGLE design)
At the start: 76 parts, among them J2 XF2L-3035-1, U0 EP4CE15E22, U4 MT48LC16M16A2, U5 OSCILLATOR5X3-PIN1-INDICATED, U6 AT25SF041-SOIC8, X1 1503_02

Commit message: add new board
Parts:
- removed C12: (no value), SparkFun-Passives:CAP0402-CAP
- C45: device SparkFun-Passives:CAP0402-CAP -> SparkFun-Passives:CAP0805
- R3, R4: device SparkFun-Passives:RESISTOR0603-RES -> SparkFun-Passives:RESISTOR0402-RES
Connections:
- removed net CKE: U0.IO@57, U4G$1.CKE
- removed net CS: U0.IO@35, U4G$1.\CS
- removed net N$12: S1.2, U0.CLK10
- new net N$16: U0.IO@9
- net /RST: no longer U0.IO@9
- net 1.0V: no longer C12.1
- net 3.3V: now also U4G$1.CKE; no longer U0.MSEL1
- net A0: now also U0.IO@26; no longer U0.IO@31
- net A1: now also U0.IO@25; no longer U0.IO@28
- net A10: now also U0.IO@27; no longer U0.IO@32
- net A2: now also U0.IO@24; no longer U0.IO@27
- net A3: now also U0.IO@23; no longer U0.IO@26
- net BA0: now also U0.IO@29; no longer U0.IO@34
- net BA1: now also U0.IO@28; no longer U0.IO@33
- net CAS: now also U0.IO@31; no longer U0.IO@39
- net CLK: now also U0.IO@57; no longer U0.IO@56
- net CLK+: now also U0.IO@20; no longer U0.IO@17
- net CLK-: now also U0.IO@21; no longer U0.IO@18
- net DQ0: now also U0.IO@40; no longer U0.IO@5
- net DQ1: now also U0.IO@43; no longer U0.IO@4
- net DQ10: now also U0.IO@53; no longer U0.IO@52
- net DQ11: now also U0.IO@52; no longer U0.IO@47
- net DQ12: now also U0.IO@51; no longer U0.IO@48
- net DQ13: now also U0.IO@50; no longer U0.IO@49
- net DQ14: now also U0.IO@49; no longer U0.IO@50
- net DQ15: now also U0.IO@48; no longer U0.IO@51
- net DQ2: now also U0.IO@44; no longer U0.IO@3
- net DQ3: now also U0.IO@45; no longer U0.IO@46
- net DQ4: now also U0.IO@46; no longer U0.IO@45
- net DQ5: now also U0.IO@47; no longer U0.IO@44
- net DQ6: now also U0.IO@35; no longer U0.IO@43
- net DQ7: now also U0.IO@34; no longer U0.IO@42
- net DQ8: now also U0.IO@55; no longer U0.IO@54
- net DQ9: now also U0.IO@54; no longer U0.IO@53
- net DQMH: now also U0.IO@56; no longer U0.IO@55
- net DQML: now also U0.IO@33; no longer U0.IO@41
- net GND: now also U4G$1.\CS; no longer C12.2, U0.MSEL0, U0.MSEL2
- net IN0+: now also U0.IO@42; no longer U0.IO@37
- net IN0-: now also U0.IO@41; no longer U0.IO@36
- net IN1+: now also U0.IO@39; no longer U0.IO@29
- net IN1-: now also U0.IO@38; no longer U0.IO@30
- net IN2+: now also U0.IO@37; no longer U0.IO@20
- net IN2-: now also U0.IO@36; no longer U0.IO@21
- net IN3+: now also U0.IO@17; no longer U0.IO@13
- net IN3-: now also U0.IO@18; no longer U0.IO@14
- net IRQ: no longer U0.CLK11
- net LED_PWM: no longer U0.IO@15
- net N$10: now also S1.2, U0.CLK11; no longer D1.C, U0.IO@11
- net RAS: now also U0.IO@30; no longer U0.IO@38
- net SCL: no longer U0.IO@8
- net SDA: no longer U0.IO@7
- net SDCD: no longer U0.CLK9
- net SDCLK: now also U0.IO@6; no longer U0.IO@22
- net SDCMD: now also U0.IO@5; no longer U0.IO@23
- net SDD0: now also U0.IO@7; no longer U0.IO@19
- net SDD1: now also U0.IO@8; no longer U0.IO@16
- net SDD2: now also U0.IO@3; no longer U0.IO@25
- net SDD3: now also U0.IO@4; no longer U0.IO@24
- net UART_RX: now also U0.IO@19; no longer U0.CLK13
- net UART_TX: now also U0.IO@22; no longer U0.IO@12
- net WE: now also U0.IO@32; no longer U0.IO@40
Other:
- moved on the sheet: /RST, GND, IRQ, J1, S1, SCL, SDA, VCC
